Commit message: 加入 Piper 关节零位偏置映射并修正 ready 姿态
- agx_arm_ctrl_single_node.py: 新增 JOINT_ZERO_OFFSETS 双向映射
  - 反馈: q_ros = q_hw - offset (硬件→ROS)
  - 命令: q_hw = q_ros + offset (ROS→硬件, 仅 MoveIt 主控制入口)
  - 真实硬件 [0.0144,0,0,0,0,1.0749] = URDF/MoveIt [0,0,0,0,0,0]
- piper.srdf.xacro: ready 改为 [0,0,0,0,0,0]
  (旧值 [0.0144,...,1.0749] 在 offset 后会导致硬件超 joint6 限位)

File: src/piper_control/config/piper.srdf.xacro (robot description, xacro)
@@ -23,10 +23,10 @@
   </group_state>
   <group_state name="ready" group="arm">
-    <joint name="joint1" value="0.0144" />
+    <joint name="joint1" value="0" />
     <joint name="joint2" value="0" />
     <joint name="joint3" value="0" />
     <joint name="joint4" value="0" />
     <joint name="joint5" value="0" />
-    <joint name="joint6" value="1.0749" />
+    <joint name="joint6" value="0" />
   </group_state>
   <!-- ======================== COLLISION DISABLES ======================== -->
